Commit message: urdf loaded

File: curdbot_description/urdf/curdbot.xacro (robot description, xacro)
@@ -3,5 +3,13 @@
 <xacro:include filename="$(find curdbot_description)/urdf/main.gazebo"/>
 <link name="base_footprint"/>
-<joint name="bf" type="fixed">
+<link name="imu_link"/>
+<joint name="imu_joint" type="fixed">
+    <axis xyz="0 0 0" />
+    <origin xyz="0 0 0.05" rpy="0 0 0" />
+    <parent link="curdbot_base" />
+    <child link="imu_link" />
+</joint>
+<!-- <link name="base_footprint"/> -->
+<joint name="basefootprint" type="fixed">
     <axis xyz="0 1 0" />
     <origin xyz="0 0 0.05" rpy="0 0 0" />

Commit message: various files changed, added laser scanner, added navigational params and some navsat/fix configs for ekf_node

File: curdbot_description/urdf/curdbot.xacro (robot description, xacro)
@@ -4,4 +4,23 @@
 <link name="base_footprint"/>
 <link name="imu_link"/>
+<link name="laser">
+<inertial>
+    <origin xyz="0.0 0.0 0.0" rpy="0 0 0" />
+    <mass value="0.3" />
+    <inertia ixx="0.3" ixy="0" ixz="0" iyy="0.2" iyz="0" izz="1.001"/>
+</inertial>
+<visual>
+    <origin xyz="0 0 0" rpy="0 0 0" />
+    <geometry>
+    <mesh filename="package://curdbot_description/meshes/dae/lidar.dae" scale="0.8 0.8 0.3" />
+    </geometry>
+</visual>
+<collision>
+<origin xyz="0 0.0 0" rpy="0 0 0" />
+    <geometry>
+    <mesh filename="package://curdbot_description/meshes/dae/lidar.dae" scale="0.8 0.8 0.3" />
+    </geometry>
+</collision>
+</link>
 <joint name="imu_joint" type="fixed">
     <axis xyz="0 0 0" />
@@ -9,4 +28,10 @@
     <parent link="curdbot_base" />
     <child link="imu_link" />
+</joint>
+<joint name="laser_joint" type="fixed">
+    <axis xyz="0 0 0"/>
+    <origin xyz="0.1 0 0.2" rpy="0 0 0" />
+    <parent link="curdbot_base" />
+    <child link="laser" />
 </joint>
 <!-- <link name="base_footprint"/> -->

Commit message: rviz config added

File: curdbot_description/urdf/curdbot.xacro (robot description, xacro)
@@ -2,5 +2,21 @@
 <robot name="curdbot" xmlns:xacro="http://www.ros.org/wiki/xacro">
 <xacro:include filename="$(find curdbot_description)/urdf/main.gazebo"/>
-<link name="base_footprint"/>
+<!-- <link name="base_footprint">
+<inertial>
+    <origin xyz="0.0 0.0 0.0" rpy="0 0 0" />
+    <mass value="28" />
+    <inertia ixx="0.3" ixy="0" ixz="0" iyy="0.2" iyz="0" izz="1.001"/>
+</inertial>
+<visual>
+    <origin xyz="0 0 0" rpy="0 0 0" />
+    <geometry>
+    </geometry>
+</visual>
+<collision>
+<origin xyz="0 0.0 0" rpy="0 0 0" />
+    <geometry>
+    </geometry>
+</collision>
+</link> -->
 <link name="imu_link"/>
 <link name="laser">
@@ -36,10 +52,10 @@
 </joint>
 <!-- <link name="base_footprint"/> -->
-<joint name="basefootprint" type="fixed">
+<!-- <joint name="basefootprint" type="fixed">
     <axis xyz="0 1 0" />
     <origin xyz="0 0 0.05" rpy="0 0 0" />
     <parent link="base_footprint" />
     <child link="curdbot_base" />
-</joint>
+</joint> -->
 <link name="curdbot_base">
 <inertial>
